File: Diagrams/Circuit Layout 2/Circuit Layout 2.kicad_sch (KiCad schematic)
At the start: 29 parts, among them J1 Barrel Jack, Q1 TIP120, Q2 TIP120, U1 LM358, U1 TRS 2-2450, U2 LM2596 3A Module, U3 HX711, U4 MPX2200GP, U5 PCF8574 Adapter, U6 1602 LCD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

Commit message: big update 12/02/2026
Parts:
- R1, R5: value R1 -> 4990
- R2, R6: value R2 -> 73
Other:
- note added: "(Equiv. R = 68)"
Changed lines of the file:
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@@
 		)
 	)
+	(text "(Equiv. R = 68)"
+		(exclude_from_sim no)
+		(at 150.876 140.208 0)
+		(effects
+			(font
+				(size 1.27 1.27)
+			)
+		)
+	)
 	(text "Pressure Sensor"
 		(exclude_from_sim no)
@@
 		)
 	)
+	(text "(Equiv. R = 68)"
+		(exclude_from_sim no)
+		(at 248.666 140.208 0)
+		(effects
+			(font
+				(size 1.27 1.27)
+			)
+		)
+	)
 	(junction
 		(at 38.1 27.94)
@@
 			)
 		)
-		(property "Value" "R2"
+		(property "Value" "73"
 			(at 195.58 132.0799 0)
 			(effects
@@
 			)
 		)
-		(property "Value" "R1"
+		(property "Value" "4990"
 			(at 97.282 119.38 0)
 			(effects
@@
 			)
 		)
-		(property "Value" "R1"
+		(property "Value" "4990"
 			(at 195.072 119.38 0)
 			(effects
@@
 			)
 		)
-		(property "Value" "R2"
+		(property "Value" "73"
 			(at 97.79 132.0799 0)
 			(effects
